Commit message: Fix ultrasonic sensor orientations and increase samples to 50 to prevent smearing

File: test_wheelchair.urdf (robot description, URDF)
Before this commit: robot wheel_chairr, 12 links, 11 joints
Joints:
- joint Fixed_U3: origin xyz=-0.0808 0.16728 -0.010721 rpy=0 0 0 -> xyz=-0.0808 0.16728 -0.010721 rpy=0 0 1.570796
- joint Fixed_US: origin xyz=-0.0807999999932945 -0.167275 -0.0107208684992432 rpy=0 0 0 -> xyz=-0.0807999999932945 -0.167275 -0.0107208684992432 rpy=0 0 -1.570796
- joint Fixed_US1: origin xyz=0.4958 0.17728 -0.017721 rpy=0 0 0 -> xyz=0.4958 0.17728 -0.017721 rpy=0 0 0.785398
- joint J_ULTRASOnic: origin xyz=0.4958 -0.17727 -0.017721 rpy=0 0 0 -> xyz=0.4958 -0.17727 -0.017721 rpy=0 0 -0.785398
